Commit message: move original config. Add xacro.

File: robot_description/urdf/mobile_kinect_manipulator.urdf (robot description, URDF)
Before this commit: robot mobile_manipulator, 14 links, 13 joints
Links:
- added link test__link, mass 0.46875; collision box size=0.15 0.05 0.05; visual box size=0.15 0.05 0.05
- added link test__link_0, mass 0.234375; collision box size=0.15 0.05 0.025; visual box size=0.15 0.05 0.025
- added link test__link_0_clone, mass 0.3125; collision box size=0.2 0.05 0.025; visual box size=0.2 0.05 0.025
- added link test__link_0_clone_0, mass 0.075; collision box size=0.06 0.05 0.02; visual box size=0.06 0.05 0.02
- link base_footprint: mass 5 -> 0
Joints:
- added joint test_link_0_joint_4: type fixed, parent test__link_0, child test__link_0_clone_0, origin xyz=-0.085    0       0.01749 rpy=-0.39713  1.57078 -0.39713
- added joint test_link_joint_2: type fixed, parent test__link, child test__link_0_clone, origin xyz=0.0625 0     0.175 rpy=-3.14159  1.57079 -3.14159
- added joint test_link_joint_3: type prismatic, parent test__link, child test__link_0, origin xyz=-0.0625  0      0.15 rpy=3.14159 1.57079 3.14159, axis 0 0 1, limit lower=0 upper=0.075 effort=-1.0 velocity=-1.0
- added joint wrist_gripper_joint: type continuous, parent top_wrist, child test__link, origin xyz=0.0 0 0.11 rpy=0 0 0, axis 0 0 1
