Commit message: reindent arm_control.yaml, change limit in arm xacro, regenerate urdf file.

File: robot_description/urdf/arm.urdf.xacro (robot description, xacro)
@@ -163,5 +163,5 @@
     <origin xyz="-0.0625  0      0.15" rpy="3.14159 1.57079 3.14159"/>
     <axis xyz="0 0 1"/>
-    <limit lower="0" upper="0.075" effort="-1.0" velocity="-1.0"/>
+    <limit lower="-0.01" upper="0.075" effort="1e6" velocity="1e6"/>
   </joint>
   <link name="test__link">

File: robot_description/urdf/mobile_kinect_manipulator.urdf (robot description, URDF)
Before this commit: robot mobile_manipulator, 18 links, 17 joints
Joints:
- joint test_link_joint_3: limit lower=0 upper=0.075 effort=-1.0 velocity=-1.0 -> lower=-0.01 upper=0.075 effort=1e6 velocity=1e6
