Commit message: Integrate darknet_ros. Update README.md. put models in postoffice+packages.world, if model is missing, installed them from forum. Regroup launch file, update yaml. TODO: depth sensor, prismatic joint, texture of packages.

File: robot_description/urdf/transmissions.urdf.xacro (robot description, xacro)
@@ -93,14 +93,5 @@
     </joint>
   </transmission>
-  <transmission name="gripper_trans" type="SimpleTransmission">
-    <type>transmission_interface/SimpleTransmission</type>
-    <actuator name="link_JOINT_3_motor">
-      <hardwareInterface>hardware_interface/PositionJointInterface</hardwareInterface>
-      <mechanicalReduction>1</mechanicalReduction>
-    </actuator>
-    <joint name="test_link_joint_3">
-      <hardwareInterface>hardware_interface/PositionJointInterface</hardwareInterface>
-    </joint>
-  </transmission>
+  <!--################################ HAND TRANSIMISSIONS ######################################-->
   <transmission name="wrist_gripper_trans" type="SimpleTransmission">
     <type>transmission_interface/SimpleTransmission</type>
@@ -113,3 +104,13 @@
     </joint>
   </transmission>
+  <transmission name="gripper_trans" type="SimpleTransmission">
+    <type>transmission_interface/SimpleTransmission</type>
+    <actuator name="test_link_motor">
+      <hardwareInterface>hardware_interface/PositionJointInterface</hardwareInterface>
+      <mechanicalReduction>1</mechanicalReduction>
+    </actuator>
+    <joint name="test_link_joint_3">
+      <hardwareInterface>hardware_interface/PositionJointInterface</hardwareInterface>
+    </joint>
+  </transmission>
 </robot>
