Commit message: update moveit config

File: mobile_manipulator_moveit_config/config/gazebo_mobile_manipulator.urdf (robot description, URDF)
Before this commit: robot mobile_manipulator, 18 links, 17 joints
Joints:
- joint test_link_joint_3: limit lower=0 upper=0.075 effort=-1.0 velocity=-1.0 -> lower=-0.01 upper=0.075 effort=1e6 velocity=1e6
